Commit message: Update project README and presentation demo assets

File: src/bumperbot_description/urdf/bumperbot.urdf.xacro (robot description, xacro)
@@ -7,4 +7,19 @@
   <!-- Include ros2_control Plugins -->
   <xacro:include filename="$(find bumperbot_description)/urdf/bumperbot_ros2_control.xacro" />
+  <material name="robot_body_blue">
+    <color rgba="0.05 0.28 0.85 1.0" />
+  </material>
+  <material name="wheel_dark">
+    <color rgba="0.02 0.02 0.025 1.0" />
+  </material>
+  <material name="caster_orange">
+    <color rgba="1.0 0.45 0.05 1.0" />
+  </material>
+  <material name="sensor_green">
+    <color rgba="0.05 0.85 0.25 1.0" />
+  </material>
+  <material name="imu_yellow">
+    <color rgba="1.0 0.82 0.10 1.0" />
+  </material>
   <link name="base_footprint"/>
   <link name="base_link">
@@ -21,4 +36,5 @@
         <mesh filename="package://bumperbot_description/meshes/base_link.STL" />
       </geometry>
+      <material name="robot_body_blue" />
     </visual>
     <collision>
@@ -47,4 +63,5 @@
         <mesh filename="package://bumperbot_description/meshes/wheel_right_link.STL" />
       </geometry>
+      <material name="wheel_dark" />
     </visual>
     <collision>
@@ -75,4 +92,5 @@
         <mesh filename="package://bumperbot_description/meshes/wheel_left_link.STL" />
       </geometry>
+      <material name="wheel_dark" />
     </visual>
     <collision>
@@ -102,4 +120,5 @@
         <mesh filename="package://bumperbot_description/meshes/caster_front_link.STL" />
       </geometry>
+      <material name="caster_orange" />
     </visual>
     <collision>
@@ -129,4 +148,5 @@
         <mesh filename="package://bumperbot_description/meshes/caster_rear_link.STL" />
       </geometry>
+      <material name="caster_orange" />
     </visual>
     <collision>
@@ -156,7 +176,5 @@
         <mesh filename="package://bumperbot_description/meshes/imu_link.STL" />
       </geometry>
-      <material name="">
-        <color rgba="0.792156862745098 0.819607843137255 0.933333333333333 1" />
-      </material>
+      <material name="imu_yellow" />
     </visual>
     <collision>
@@ -186,7 +204,5 @@
         <box size="0.01 0.01 0.01" />
       </geometry>
-      <material name="">
-        <color rgba="0.2 0.8 0.2 1.0" />
-      </material>
+      <material name="sensor_green" />
     </visual>
     <collision>

File: src/bumperbot_description/urdf/bumperbot_gazebo.xacro (robot description, xacro)
@@ -1,6 +1,14 @@
 <?xml version="1.0"?>
 <robot name="bumperbot" xmlns:xacro="http://ros.org/wiki/xacro">
+  <gazebo reference="base_link">
+    <material>Gazebo/Blue</material>
+    <ambient>0.05 0.28 0.85 1.0</ambient>
+    <diffuse>0.05 0.28 0.85 1.0</diffuse>
+  </gazebo>
   <!-- Wheels -->
   <gazebo reference="wheel_left_link">
+    <material>Gazebo/Black</material>
+    <ambient>0.02 0.02 0.025 1.0</ambient>
+    <diffuse>0.02 0.02 0.025 1.0</diffuse>
     <mu1>1000000000000000.0</mu1>
     <mu2>1000000000000000.0</mu2>
@@ -12,4 +20,7 @@
   </gazebo>
   <gazebo reference="wheel_right_link">
+    <material>Gazebo/Black</material>
+    <ambient>0.02 0.02 0.025 1.0</ambient>
+    <diffuse>0.02 0.02 0.025 1.0</diffuse>
     <mu1>1000000000000000.0</mu1>
     <mu2>1000000000000000.0</mu2>
@@ -22,4 +33,7 @@
   <!-- Caster Wheels -->
   <gazebo reference="caster_rear_link">
+    <material>Gazebo/Orange</material>
+    <ambient>1.0 0.45 0.05 1.0</ambient>
+    <diffuse>1.0 0.45 0.05 1.0</diffuse>
     <mu1>0.1</mu1>
     <mu2>0.1</mu2>
@@ -30,4 +44,7 @@
   </gazebo>
   <gazebo reference="caster_front_link">
+    <material>Gazebo/Orange</material>
+    <ambient>1.0 0.45 0.05 1.0</ambient>
+    <diffuse>1.0 0.45 0.05 1.0</diffuse>
     <mu1>0.1</mu1>
     <mu2>0.1</mu2>
@@ -56,4 +73,7 @@
   <!-- IMU -->
   <gazebo reference="imu_link">
+    <material>Gazebo/Yellow</material>
+    <ambient>1.0 0.82 0.10 1.0</ambient>
+    <diffuse>1.0 0.82 0.10 1.0</diffuse>
     <sensor name="imu" type="imu">
         <always_on>true</always_on>
@@ -107,4 +127,7 @@
    <!-- GPS -->
   <gazebo reference="gps_link">
+    <material>Gazebo/Green</material>
+    <ambient>0.05 0.85 0.25 1.0</ambient>
+    <diffuse>0.05 0.85 0.25 1.0</diffuse>
     <sensor name="gps_sensor" type="navsat">
       <always_on>true</always_on>
